File: os9_mmu/os9_mmu.kicad_sch (KiCad schematic)
At the start: 18 parts, among them U1 74LS257, U2 74LS157, U3 74LS273, U4 74LS04, U5 74LS02, U6 6809E

Commit message: MMU adjustments
-adjusted power trace widths
-reintroduced solder mask layer - was absence to give board a vintage look but makes silkscreen prints impossible
-fixed license links in drawing sheets to match board prints, readme and project
Other:
- note added: "+5V"
- note added: "21"
- note added: "22"
- note added: "23"
- note added: "24"
- note added: "25"
- note added: "26"
- note added: "27"
- note added: "28"
- note added: "29"
- note added: "30"
- note added: "31"
- note added: "32"
- note added: "33"
- note added: "34"
- note added: "35"
- note added: "36"
- note added: "37"
- note added: "38"
- note added: "39"
- note added: "40"
- note added: "D0"
- note added: "D1"
- note added: "D2"
- note added: "D3"
- note added: "D4"
- note added: "D5"
- note added: "D6"
- note added: "D7"
- note added: "GND"
- note added: "MR"
- note added: "NC"
- moved on the sheet: JC1, JL1, JL2, JP2, JR1, JR2, U1, U2, U3, U4A, U4C, U4D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
